File: pcb/facewhisperer.brd (EAGLE design)
At the start: 100 x 80 mm, 15 parts, among them IC1 XMEGA128D4, J1 CWTIO-20PIN, J2 VUSB IN, J3 USB-A-H, J5 CLK3, J6 RESET, U1 MAX3421ESMD, U2 NC7WZ14, X1 CLK1, X2 CLK2

Commit message: First rev of the PCB design
Parts:
- added C2, C3, C4, C5: 100n, SparkFun-Passives:0805
- added C6: 1u, SparkFun-Passives:0805
- added F1: PTC 2A, SparkFun-PowerIC:PTC-1206-WIDE
- added H1, H2, H3, H4: MOUNT-HOLE3.2, holes:3,2
- added LED1: Power, adafruit:1206
- added LED2: Reset, adafruit:1206
- added LED3: VBUS, adafruit:1206
- added LED4: PA5, adafruit:1206
- added LED5: PA6, adafruit:1206
- added R10, R11, R4, R6, R7: 1k, SparkFun-Passives:0805
- added R2, R5: 100, SparkFun-Passives:0805
- added R3: 10k, SparkFun-Passives:0805
- added R8, R9: 33, SparkFun-Passives:0805
- U1: device SparkFun-DigitalIC:TQFP32-5MM -> SparkFun-DigitalIC:TQFP32-5MM-MILLABLE
- U2: device fairchild-semi:SC70-6 -> fairchild-semi:SC70-6-MILLABLE
- moved J6 125.0 mm to (54.6, 54.6), turned to 270 degrees
- moved FRAME1 121.2 mm to (44.5, 58.4)
- moved X2 114.8 mm to (38.1, 81.3), turned to 270 degrees
- moved X1 112.0 mm to (55.9, 64.8), turned to 180 degrees
- moved J2 95.3 mm to (58.4, 17.8), turned to 90 degrees
- moved U2 93.3 mm to (36.8, 63.5), turned to 270 degrees
- moved J5 79.2 mm to (35.6, 73.7)
- moved Q1 70.4 mm to (48.3, 52.1), turned to 270 degrees
- moved C1 61.2 mm to (35.3, 67.1), turned to 180 degrees
- moved R1 57.2 mm to (41.9, 62.9)
- moved J3 43.4 mm to (48.3, 36.8)
- moved IC1 41.5 mm to (27.9, 21.1), turned to 180 degrees
- moved J4 38.9 mm to (39.4, 33.0)
- moved U1 29.2 mm to (27.9, 37.6)
- moved J1 26.5 mm to (8.89, 30.5)
Connections:
- removed net AVCC: IC1.39
- removed net VCC: IC1.9
- removed net VCC1: IC1.19
- removed net VCC2: IC1.31
- new net N$10: LED3.A, R7.1
- new net N$11: R9.2, U1.20
- new net N$12: R8.2, U1.21
- new net N$13: F1.1, J2.PWR
- new net N$14: LED4.A, R10.1
- new net N$15: LED5.A, R11.1
- new net N$16: IC1.2, LED5.C
- new net N$17: IC1.1, LED4.C
- new net N$4: R5.2, U1.24
- new net N$6: LED2.A, R4.2
- new net N$7: IC1.37, R2.2
- new net N$9: LED1.A, R6.1
- new net PDI_CLK: IC1.35, J1.13, R3.1
- new net PDI_DATA: IC1.34, J1.15
- new net TIO1: IC1.13, J1.10
- new net TIO2: IC1.12, J1.12
- new net TIO3: IC1.41, J1.14
- new net TIO4: IC1.40, J1.16
- new net USB_GPX: IC1.10, U1.17
- new net USB_IRQ: IC1.6, U1.18
- new net USB_MISO: IC1.16, U1.15
- new net USB_MOSI: IC1.15, U1.16
- new net USB_RESET: IC1.11, U1.12
- new net USB_SCK: IC1.17, U1.13
- new net USB_SS: IC1.14, U1.14
- net 3.3V: now also C2.1, C3.1, C4.1, C5.1, C6.1, IC1.19, IC1.31, IC1.39, IC1.9, J1.8, R10.2, R11.2, R3.2, R6.2, U1.2, U1.23
- net CLK12: now also J1.6, R2.1, R5.1
- net D+: now also R8.1
- net D-: now also R9.1
- net GND: now also C2.2, C3.2, C4.2, C5.2, C6.2, J1.17, J1.19, J1.2, LED1.C, LED2.C, LED3.C, U1.19, U1.3
- net N$5: now also F1.2, R7.2; no longer J2.PWR
- net RESET_GATE: now also IC1.3, R4.1
Routing:
- net GND: track 0.00 -> 414.7 mm
- net 3.3V: track 0.00 -> 242.7 mm, vias 0 -> 3
- net CLK12: track 0.00 -> 121.1 mm, vias 0 -> 3
- net RESET_GATE: track 0.00 -> 57.6 mm, vias 0 -> 2
- net N$5: track 0.00 -> 42.0 mm
- net PDI_CLK: track 0.00 -> 36.6 mm
- net N$3: track 0.00 -> 32.0 mm
- net TIO3: track 0.00 -> 31.7 mm, vias 0 -> 1
- net TIO4: track 0.00 -> 31.2 mm, vias 0 -> 1
- net PDI_DATA: track 0.00 -> 29.1 mm
- net TIO2: track 0.00 -> 26.2 mm, vias 0 -> 1
- net N$16: track 0.00 -> 25.6 mm
- net TIO1: track 0.00 -> 25.2 mm, vias 0 -> 1
- net USB_IRQ: track 0.00 -> 23.5 mm, vias 0 -> 2
- net USB_RESET: track 0.00 -> 17.2 mm
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- added copper zone on layer 1, net GND
- added copper zone on layer 16, net GND
Other:
- board size 100 x 80 mm -> 58.4 x 83.8 mm

Commit message: Add a sync input for use with analog comparator
Parts:
- added J7: SYNCIN, SparkFun-Connectors:1X03_LOCK_LONGPADS
Connections:
- new net SYNC_IN: IC1.44, J7.2
- net GND: now also J7.1, J7.3
Changed lines of the file:
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@@
 <element name="H4" library="holes" package="3,2" value="MOUNT-HOLE3.2" x="6.35" y="77.47"/>
 <element name="F1" library="SparkFun-PowerIC" package="PTC-1206-WIDE" value="PTC 2A" x="43.18" y="8.89" rot="R180"/>
+<element name="J7" library="SparkFun-Connectors" package="1X03_LOCK_LONGPADS" value="SYNCIN" x="1.778" y="-3.81"/>
 </elements>
 <signals>
@@
 <vertex x="0" y="0"/>
 </polygon>
+<contactref element="J7" pad="3"/>
+<contactref element="J7" pad="1"/>
+<wire x1="6.858" y1="-3.81" x2="9.144" y2="15.748" width="0" layer="19" extent="1-1"/>
+<wire x1="1.778" y1="-3.81" x2="6.858" y2="-3.81" width="0" layer="19" extent="1-1"/>
 </signal>
 <signal name="3.3V">
@@
 <wire x1="44.72" y1="8.89" x2="44.72" y2="17.78" width="0.8128" layer="1"/>
 </signal>
+<signal name="SYNC_IN">
+<contactref element="IC1" pad="44"/>
+<contactref element="J7" pad="2"/>
+<wire x1="4.318" y1="-4.064" x2="31.94" y2="15.282" width="0" layer="19" extent="1-1"/>
+</signal>
 </signals>
